Commit message: feat: Added gripper models

File: pro_arm_description/urdf/pro_arm.urdf.xacro (robot description, xacro)
@@ -1,4 +1,4 @@
 <?xml version="1.0"?>
-<!-- URDF for PRO 5DoF/6DoF Arms -->
+<!-- URDF for PRO Arms -->
 <robot xmlns:xacro="http://wiki.ros.org/xacro" name="$(arg name)">
   <!--                   -->
@@ -14,4 +14,8 @@
   <!-- Parameter to select size version -->
   <xacro:arg name="size" default="550"/>
+  <!-- Parameter to select gripper model -->
+  <xacro:arg name="gripper" default="none"/>
+  <!-- Parameter to select finger separation model -->
+  <xacro:arg name="finger" default="40"/>
   <!-- Name of the robot (mandatory) -->
   <xacro:arg name="name" default="pro_arm"/>
@@ -21,8 +25,4 @@
   <!-- Flag to enable collision geometry for manipulator's arm -->
   <xacro:arg name="collision" default="true"/>
-  <!-- Flag to enable safety limits controllers on manipulator joints -->
-  <!-- <xacro:arg name="safety_limits" default="false"/> -->
-  <!-- Lower and upper margin for position limits of all safety controllers (1 deg)-->
-  <!-- <xacro:arg name="safety_position_margin" default="0.17453293"/> -->
   <!-- Flag to enable ros2 controllers for manipulator -->
   <xacro:arg name="ros2_control" default="true"/>
@@ -42,7 +42,4 @@
   <xacro:property name="origin_xyz" value="0 0 0"/>
   <xacro:property name="origin_rpy" value="0 0 0"/>
-  <!-- Offset of gripper with respect to wrist flange -->
-  <!-- <xacro:property name="gripper_offset_xyz" value="0 0 0"/>
-  <xacro:property name="gripper_offset_rpy" value="0 0 0"/> -->
   <!--       -->
   <!-- Robot -->
@@ -83,19 +80,43 @@
   </xacro:if>
   <!-- Gripper -->
-  <!-- <xacro:include filename="$(find pro_arm_description)/urdf/pro_gripper_4dof.xacro"/>
-  <xacro:gripper_5dof
-    pro_gripper="${prefix_arm}gripper_5dof"
+  <xacro:if value="${'$(arg gripper)' == 'none'}">
+  <xacro:include filename="$(find pro_arm_description)/urdf/no_gripper.xacro"/>
+  <xacro:no_gripper
+    pro_gripper="${'$(arg gripper)'}"
     prefix="${prefix_arm}"
-    origin_xyz="${gripper_offset_xyz}"
-    origin_rpy="${gripper_offset_rpy}"
+    gripper="${'$(arg gripper)'}"
+    size="${'$(arg size)'}"
     collision="$(arg collision)"
-    safety_limits="$(arg safety_limits)"
-    safety_position_margin="$(arg safety_position_margin)"
-    safety_k_position="$(arg safety_k_position)"
-    safety_k_velocity="$(arg safety_k_velocity)"
     ros2_control="$(arg ros2_control)"
     ros2_control_plugin="$(arg ros2_control_plugin)"
     gazebo_preserve_fixed_joint="$(arg gazebo_preserve_fixed_joint)"
-  /> -->
+  />
+  </xacro:if>
+  <xacro:if value="${'$(arg gripper)' == 'pge_5040'}">
+  <xacro:include filename="$(find pro_arm_description)/urdf/dh_gripper_pge_5040.xacro"/>
+  <xacro:gripper_pge_5040
+    pro_gripper="${'$(arg gripper)'}"
+    prefix="${prefix_arm}"
+    gripper="${'$(arg gripper)'}"
+    finger="${'$(arg finger)'}"
+    collision="$(arg collision)"
+    ros2_control="$(arg ros2_control)"
+    ros2_control_plugin="$(arg ros2_control_plugin)"
+    gazebo_preserve_fixed_joint="$(arg gazebo_preserve_fixed_joint)"
+  />
+  </xacro:if>
+  <xacro:if value="${'$(arg gripper)' == 'cge_1010'}">
+  <xacro:include filename="$(find pro_arm_description)/urdf/dh_gripper_cge_1010.xacro"/>
+  <xacro:gripper_cge_1010
+    pro_gripper="${'$(arg gripper)'}"
+    prefix="${prefix_arm}"
+    gripper="${'$(arg gripper)'}"
+    finger="${'$(arg finger)'}"
+    collision="$(arg collision)"
+    ros2_control="$(arg ros2_control)"
+    ros2_control_plugin="$(arg ros2_control_plugin)"
+    gazebo_preserve_fixed_joint="$(arg gazebo_preserve_fixed_joint)"
+  />
+  </xacro:if>
   <!-- Gazebo - ROS 2 control -->
   <xacro:if value="$(arg ros2_control)">

File: pro_arm_description/urdf/pro_arm_550.xacro (robot description, xacro)
@@ -34,21 +34,21 @@
   <xacro:property name="base_joint_type" value="fixed"/>
   <xacro:property name="joint_1_type" value="revolute"/>
-  <xacro:property name="joint_1_origin_xyz" value="0 0 0.0315"/>
-  <xacro:property name="joint_1_origin_rpy" value="1.5708 1.5708 0"/>
-  <xacro:property name="joint_1_axis_xyz" value="1 0 0"/>
+  <xacro:property name="joint_1_origin_xyz" value="0 0 0.0065"/>
+  <xacro:property name="joint_1_origin_rpy" value="1.5708 0 0"/>
+  <xacro:property name="joint_1_axis_xyz" value="0 -1 0"/>
   <xacro:property name="joint_1_lower_limit" value="${-pi}"/>
   <xacro:property name="joint_1_upper_limit" value="${pi}"/>
   <xacro:property name="joint_2_type" value="revolute"/>
-  <xacro:property name="joint_2_origin_xyz" value="-0.05 0 -0.045583"/>
-  <xacro:property name="joint_2_origin_rpy" value="0.7854 1.5708 1.5708"/>
-  <xacro:property name="joint_2_axis_xyz" value="1 0 0"/>
-  <xacro:property name="joint_2_lower_limit" value="${-pi/2}"/>
-  <xacro:property name="joint_2_upper_limit" value="${pi/2}"/>
+  <xacro:property name="joint_2_origin_xyz" value="0.070003 0.075 0"/>
+  <xacro:property name="joint_2_origin_rpy" value="0 0 0"/>
+  <xacro:property name="joint_2_axis_xyz" value="-1 0 0"/>
+  <xacro:property name="joint_2_lower_limit" value="${-pi}"/>
+  <xacro:property name="joint_2_upper_limit" value="${pi}"/>
   <xacro:property name="joint_3_type" value="revolute"/>
-  <xacro:property name="joint_3_origin_xyz" value="0 0.1591 -0.1591"/>
-  <xacro:property name="joint_3_origin_rpy" value="1.5511 0 0"/>
+  <xacro:property name="joint_3_origin_xyz" value="-0.033961 0.225 0"/>
+  <xacro:property name="joint_3_origin_rpy" value="0 0 0"/>
   <xacro:property name="joint_3_axis_xyz" value="1 0 0"/>
-  <xacro:property name="joint_3_lower_limit" value="${-120*pi/180}"/>
-  <xacro:property name="joint_3_upper_limit" value="${120*pi/180}"/>
+  <xacro:property name="joint_3_lower_limit" value="${-pi}"/>
+  <xacro:property name="joint_3_upper_limit" value="${pi}"/>
   <xacro:if value="${'$(arg dof)' == '5'}">
     <xacro:property name="joint_4_type" value="fixed"/>
@@ -61,21 +61,13 @@
     <xacro:property name="joint_4_upper_limit" value="${pi}"/>
   </xacro:if>
-  <xacro:property name="joint_4_origin_xyz" value="-0.05 0 0"/>
+  <xacro:property name="joint_4_origin_xyz" value="-0.036042 0.073 0"/>
   <xacro:property name="joint_4_origin_rpy" value="0 0 0"/>
-  <xacro:property name="joint_4_axis_xyz" value="0 0.69305 0.72089"/>
+  <xacro:property name="joint_4_axis_xyz" value="0 -1 0"/>
   <xacro:property name="joint_5_type" value="revolute"/>
-  <xacro:property name="joint_5_origin_xyz" value="0.048417 -0.17257 -0.1795"/>
-  <xacro:property name="joint_5_origin_rpy" value="0.80509 0 0"/>
-  <xacro:property name="joint_5_axis_xyz" value="1 0 0"/>
+  <xacro:property name="joint_5_origin_xyz" value="0.088958 0.175 0"/>
+  <xacro:property name="joint_5_origin_rpy" value="0 0 0"/>
+  <xacro:property name="joint_5_axis_xyz" value="-1 0 0"/>
   <xacro:property name="joint_5_lower_limit" value="${-pi}"/>
   <xacro:property name="joint_5_upper_limit" value="${pi}"/>
-  <xacro:property name="joint_6_type" value="revolute"/>
-  <xacro:property name="joint_6_origin_xyz" value="0.076 0.048 0"/>
-  <xacro:property name="joint_6_origin_rpy" value="1.5708 1.5708 1.5708"/>
-  <xacro:property name="joint_6_axis_xyz" value="0 1 0"/>
-  <xacro:property name="joint_6_lower_limit" value="${-pi}"/>
-  <xacro:property name="joint_6_upper_limit" value="${pi}"/>
-  <xacro:property name="ee_origin_xyz" value="0 0.025 0"/>
-  <xacro:property name="ee_origin_rpy" value="0 0 0"/>
     <!--       -->
     <!-- Macro -->
@@ -246,39 +238,4 @@
     mu="${mu}"
     />
-    <!-- 6 -->
-    <xacro:pro_arm_joint_
-    parent="${prefix}link_5"
-    child="${prefix}link_6"
-    joint_name="${prefix}joint_6"
-    joint_type="${joint_6_type}"
-    joint_origin_xyz="${joint_6_origin_xyz}"
-    joint_origin_rpy="${joint_6_origin_rpy}"
-    joint_axis_xyz="${joint_6_axis_xyz}"
-    joint_lower_limit="${joint_6_lower_limit}"
-    joint_upper_limit="${joint_6_upper_limit}"
-    joint_velocity_limit="${l1_velocity_limit}"
-    joint_torque_limit="${l1_torque_limit}"
-    joint_damping="${l1_damping}"
-    joint_friction="${l1_friction}"
-    safety_limits="${safety_limits}"
-    safety_position_margin="${safety_position_margin}"
-    safety_k_position="${l1_safety_k_position}"
-    safety_k_velocity="${l1_safety_k_velocity}"
-    gazebo_preserve_fixed_joint="${gazebo_preserve_fixed_joint}"
-    />
-    <xacro:pro_arm_link
-    link_name="${prefix}link_6"
-    size="550"
-    collision="${collision}"
-    mu="${mu}"
-    />
-    <!-- End effector -->
-    <xacro:pro_arm_virtual_link
-    parent="${prefix}link_6"
-    link_name="${prefix}ee"
-    joint_origin_xyz="${ee_origin_xyz}"
-    joint_origin_rpy="${ee_origin_rpy}"
-    gazebo_preserve_fixed_joint="${gazebo_preserve_fixed_joint}"
-    />
      <!-- ROS 2 control -->
     <xacro:if value="${ros2_control}">

File: pro_arm_description/urdf/pro_arm_900.xacro (robot description, xacro)
@@ -43,21 +43,21 @@
   <xacro:property name="base_joint_type" value="fixed"/>
   <xacro:property name="joint_1_type" value="revolute"/>
-  <xacro:property name="joint_1_origin_xyz" value="0 0 0.042"/>
-  <xacro:property name="joint_1_origin_rpy" value="1.5708 1.5708 0"/>
-  <xacro:property name="joint_1_axis_xyz" value="1 0 0"/>
+  <xacro:property name="joint_1_origin_xyz" value="0 0 0"/>
+  <xacro:property name="joint_1_origin_rpy" value="1.5707963267949 0 0.0428232118686817"/>
+  <xacro:property name="joint_1_axis_xyz" value="0 -1 0"/>
   <xacro:property name="joint_1_lower_limit" value="${-pi}"/>
   <xacro:property name="joint_1_upper_limit" value="${pi}"/>
   <xacro:property name="joint_2_type" value="revolute"/>
-  <xacro:property name="joint_2_origin_xyz" value="-0.075 0 -0.063583"/>
-  <xacro:property name="joint_2_origin_rpy" value="-1.9695 1.5708 -0.87159"/>
-  <xacro:property name="joint_2_axis_xyz" value="1 0 0"/>
-  <xacro:property name="joint_2_lower_limit" value="${-pi/2}"/>
-  <xacro:property name="joint_2_upper_limit" value="${pi/2}"/>
+  <xacro:property name="joint_2_origin_xyz" value="0.0753209069561978 0.108 0"/>
+  <xacro:property name="joint_2_origin_rpy" value="-0.004865934294438 0 0"/>
+  <xacro:property name="joint_2_axis_xyz" value="-1 0 0"/>
+  <xacro:property name="joint_2_lower_limit" value="${-pi}"/>
+  <xacro:property name="joint_2_upper_limit" value="${pi}"/>
   <xacro:property name="joint_3_type" value="revolute"/>
-  <xacro:property name="joint_3_origin_xyz" value="0 0.36722 -0.18789"/>
-  <xacro:property name="joint_3_origin_rpy" value="0.31248 0 0"/>
+  <xacro:property name="joint_3_origin_xyz" value="0 0.412499999999363 0"/>
+  <xacro:property name="joint_3_origin_rpy" value="-1.56593039250046 0 0"/>
   <xacro:property name="joint_3_axis_xyz" value="1 0 0"/>
-  <xacro:property name="joint_3_lower_limit" value="${-120*pi/180}"/>
-  <xacro:property name="joint_3_upper_limit" value="${120*pi/180}"/>
+  <xacro:property name="joint_3_lower_limit" value="${-pi}"/>
+  <xacro:property name="joint_3_upper_limit" value="${pi}"/>
   <xacro:if value="${'$(arg dof)' == '5'}">
     <xacro:property name="joint_4_type" value="fixed"/>
@@ -70,21 +70,13 @@
     <xacro:property name="joint_4_upper_limit" value="${pi}"/>
   </xacro:if>
-  <xacro:property name="joint_4_origin_xyz" value="-0.024583 0.0026942 -0.0026942"/>
-  <xacro:property name="joint_4_origin_rpy" value="0 0 0"/>
-  <xacro:property name="joint_4_axis_xyz" value="0 0.70711 -0.70711"/>
+  <xacro:property name="joint_4_origin_xyz" value="-0.0253209069561977 0 0.075"/>
+  <xacro:property name="joint_4_origin_rpy" value="1.5707963267949 0 0"/>
+  <xacro:property name="joint_4_axis_xyz" value="0 -1 0"/>
   <xacro:property name="joint_5_type" value="revolute"/>
-  <xacro:property name="joint_5_origin_xyz" value="0.048 0.28828 -0.28828"/>
-  <xacro:property name="joint_5_origin_rpy" value="-0.7854 0 0"/>
-  <xacro:property name="joint_5_axis_xyz" value="1 0 0"/>
+  <xacro:property name="joint_5_origin_xyz" value="0.0751686090232449 0.337500000000057 0"/>
+  <xacro:property name="joint_5_origin_rpy" value="0 0 0"/>
+  <xacro:property name="joint_5_axis_xyz" value="-1 0 0"/>
   <xacro:property name="joint_5_lower_limit" value="${-pi}"/>
   <xacro:property name="joint_5_upper_limit" value="${pi}"/>
-  <xacro:property name="joint_6_type" value="revolute"/>
-  <xacro:property name="joint_6_origin_xyz" value="0.076 -0.048 0"/>
-  <xacro:property name="joint_6_origin_rpy" value="3.1416 -1.5454 3.1416"/>
-  <xacro:property name="joint_6_axis_xyz" value="0 1 0"/>
-  <xacro:property name="joint_6_lower_limit" value="${-pi}"/>
-  <xacro:property name="joint_6_upper_limit" value="${pi}"/>
-  <xacro:property name="ee_origin_xyz" value="0 -0.025 0"/>
-  <xacro:property name="ee_origin_rpy" value="0 0 0"/>
     <!--       -->
     <!-- Macro -->
@@ -255,39 +247,4 @@
     mu="${mu}"
     />
-    <!-- 6 -->
-    <xacro:pro_arm_joint_
-    parent="${prefix}link_5"
-    child="${prefix}link_6"
-    joint_name="${prefix}joint_6"
-    joint_type="${joint_6_type}"
-    joint_origin_xyz="${joint_6_origin_xyz}"
-    joint_origin_rpy="${joint_6_origin_rpy}"
-    joint_axis_xyz="${joint_6_axis_xyz}"
-    joint_lower_limit="${joint_6_lower_limit}"
-    joint_upper_limit="${joint_6_upper_limit}"
-    joint_velocity_limit="${l1_velocity_limit}"
-    joint_torque_limit="${l1_torque_limit}"
-    joint_damping="${l1_damping}"
-    joint_friction="${l1_friction}"
-    safety_limits="${safety_limits}"
-    safety_position_margin="${safety_position_margin}"
-    safety_k_position="${l1_safety_k_position}"
-    safety_k_velocity="${l1_safety_k_velocity}"
-    gazebo_preserve_fixed_joint="${gazebo_preserve_fixed_joint}"
-    />
-    <xacro:pro_arm_link
-    link_name="${prefix}link_6"
-    size="900"
-    collision="${collision}"
-    mu="${mu}"
-    />
-    <!-- End effector -->
-    <xacro:pro_arm_virtual_link
-    parent="${prefix}link_6"
-    link_name="${prefix}ee"
-    joint_origin_xyz="${ee_origin_xyz}"
-    joint_origin_rpy="${ee_origin_rpy}"
-    gazebo_preserve_fixed_joint="${gazebo_preserve_fixed_joint}"
-    />
      <!-- ROS 2 control -->
     <xacro:if value="${ros2_control}">
