Commit message: fix: Adjusted max speeds

File: pro_arm_description/urdf/pro_arm_550.xacro (robot description, xacro)
@@ -15,5 +15,5 @@
   <!--    Servo   -->
   <xacro:property name="l1_torque_limit" value="19"/>
-  <xacro:property name="l1_velocity_limit" value="0.78540"/>
+  <xacro:property name="l1_velocity_limit" value="1.31"/>
   <xacro:property name="l1_damping" value="0.1"/>
   <xacro:property name="l1_friction" value="0.5"/>
@@ -24,5 +24,5 @@
   <!--   Servo    -->
   <xacro:property name="s1_torque_limit" value="54"/>
-  <xacro:property name="s1_velocity_limit" value="0.78540"/>
+  <xacro:property name="s1_velocity_limit" value="1.57"/>
   <xacro:property name="s1_damping" value="0.1"/>
   <xacro:property name="s1_friction" value="0.5"/>
@@ -85,4 +85,5 @@
       ros2_control:=true
       ros2_control_plugin:=fake
+      size:=550
       gazebo_preserve_fixed_joint:=false
     ">

File: pro_arm_description/urdf/pro_arm_900.xacro (robot description, xacro)
@@ -15,5 +15,5 @@
   <!--    Servo   -->
   <xacro:property name="l1_torque_limit" value="19"/>
-  <xacro:property name="l1_velocity_limit" value="0.78540"/>
+  <xacro:property name="l1_velocity_limit" value="1.31"/>
   <xacro:property name="l1_damping" value="0.1"/>
   <xacro:property name="l1_friction" value="0.5"/>
@@ -24,5 +24,5 @@
   <!--   Servo    -->
   <xacro:property name="s1_torque_limit" value="54"/>
-  <xacro:property name="s1_velocity_limit" value="0.78540"/>
+  <xacro:property name="s1_velocity_limit" value="1.57"/>
   <xacro:property name="s1_damping" value="0.1"/>
   <xacro:property name="s1_friction" value="0.5"/>
@@ -33,5 +33,5 @@
   <!--    Servo   -->
   <xacro:property name="m1_torque_limit" value="130"/>
-  <xacro:property name="m1_velocity_limit" value="1.57"/>
+  <xacro:property name="m1_velocity_limit" value="1.13"/>
   <xacro:property name="m1_damping" value="0.1"/>
   <xacro:property name="m1_friction" value="0.5"/>
@@ -94,4 +94,5 @@
       ros2_control:=true
       ros2_control_plugin:=fake
+      size:=900
       gazebo_preserve_fixed_joint:=false
     ">
